Commit message: a version can work but not so stable

File: je_software/urdf/L_JEARM/L_JEARM.urdf (robot description, URDF)
Before this commit: robot RH_JEARM, 8 links, 7 joints
Links:
- link Link1: mass 0.159032417486965 -> 0.15903
- link Link2: mass 0.243793701990545 -> 0.24379
- link Link3: mass 0.249547645812497 -> 0.24955
- link Link4: mass 0.140360397584585 -> 0.14036
- link Link5: mass 0.203459403127019 -> 0.20346
- link Link6: mass 0.139511938718154 -> 0.13951
- link Link7: mass 0.369145497401337 -> 0.36915
Joints:
- joint joint1: limit lower=-31.4 upper=31.4 effort=100 velocity=31.4 -> lower=-5.14 upper=5.14 effort=100 velocity=3.14; origin xyz=-0.0445 -0.2126 0.9008 rpy=1.5708 -1.5708 0 -> xyz=0 0 0 rpy=0 0 0
- joint joint2: limit lower=-31.4 upper=31.4 effort=100 velocity=31.4 -> lower=-2.96 upper=2.96 effort=100 velocity=3.14
- joint joint3: limit lower=-31.4 upper=31.4 effort=100 velocity=31.4 -> lower=-2.96 upper=2.96 effort=100 velocity=3.14
- joint joint4: limit lower=-31.4 upper=31.4 effort=100 velocity=31.4 -> lower=-2.27 upper=1.8 effort=100 velocity=3.14
- joint joint5: limit lower=-31.4 upper=31.4 effort=100 velocity=31.4 -> lower=-2.96 upper=2.96 effort=100 velocity=3.14
- joint joint6: limit lower=-31.4 upper=31.4 effort=100 velocity=31.4 -> lower=-1.6 upper=1.55 effort=100 velocity=3.14
- joint joint7: limit lower=-31.4 upper=31.4 effort=100 velocity=31.4 -> lower=-2.96 upper=2.96 effort=100 velocity=3.14

File: je_software/urdf/R_JEARM/R_JEARM.urdf (robot description, URDF)
Before this commit: robot RH_JEARM, 8 links, 7 joints
Links:
- link Link1: mass 0.159032417495047 -> 0.15903
- link Link2: mass 0.243793701990545 -> 0.24379
- link Link3: mass 0.249547645812502 -> 0.24955
- link Link4: mass 0.140360397584585 -> 0.14036
- link Link5: mass 0.203459403127014 -> 0.20346
- link Link6: mass 0.139511938718152 -> 0.13951
- link Link7: mass 0.369150471437428 -> 0.36915
- link base_link: mass 34.2155433013561 -> 34.216
Joints:
- joint joint1: limit lower=-31.4 upper=31.4 effort=100 velocity=31.4 -> lower=-5.14 upper=5.14 effort=100 velocity=3.14; origin xyz=-0.0445 0.2126 0.9008 rpy=1.5708 -1.5708 0 -> xyz=0 0 0 rpy=0 0 0
- joint joint2: limit lower=-31.4 upper=31.4 effort=100 velocity=31.4 -> lower=-1.86 upper=1.82 effort=100 velocity=3.14
- joint joint3: limit lower=-31.4 upper=31.4 effort=100 velocity=31.4 -> lower=-2.96 upper=2.96 effort=100 velocity=3.14
- joint joint4: limit lower=-31.4 upper=31.4 effort=100 velocity=31.4 -> lower=-2.27 upper=1.8 effort=100 velocity=3.14
- joint joint5: limit lower=-31.4 upper=31.4 effort=100 velocity=31.4 -> lower=-2.96 upper=2.96 effort=100 velocity=3.14
- joint joint6: limit lower=-31.4 upper=31.4 effort=100 velocity=31.4 -> lower=-1.6 upper=1.55 effort=100 velocity=3.14
- joint joint7: limit lower=-31.4 upper=31.4 effort=100 velocity=31.4 -> lower=-2.96 upper=2.96 effort=100 velocity=3.14
